Commit message: Added Minitaur with sensor head

File: minitaur_description/urdf/minitaur.urdf (robot description, URDF)
Before this commit: robot minitaur, 39 links, 38 joints
Links:
- link motor_back_leftL_link: geometry collision cylinder length=0.021 radius=0.0425; visual mesh filename=package://minitaur_description/meshes/tmotor3.obj scale=1.0 1.0 1.0
- link motor_back_leftR_link: geometry collision cylinder length=0.021 radius=0.0425; visual mesh filename=package://minitaur_description/meshes/tmotor3.obj scale=1.0 1.0 1.0
- link motor_back_rightL_link: geometry collision cylinder length=0.021 radius=0.0425; visual mesh filename=package://minitaur_description/meshes/tmotor3.obj scale=1.0 1.0 1.0
- link motor_back_rightR_link: geometry collision cylinder length=0.021 radius=0.0425; visual mesh filename=package://minitaur_description/meshes/tmotor3.obj scale=1.0 1.0 1.0
- link motor_front_leftL_link: geometry collision cylinder length=0.021 radius=0.0425; visual mesh filename=package://minitaur_description/meshes/tmotor3.obj scale=1.0 1.0 1.0
- link motor_front_leftR_link: geometry collision cylinder length=0.021 radius=0.0425; visual mesh filename=package://minitaur_description/meshes/tmotor3.obj scale=1.0 1.0 1.0
- link motor_front_rightL_link: geometry collision cylinder length=0.021 radius=0.0425; visual mesh filename=package://minitaur_description/meshes/tmotor3.obj scale=1.0 1.0 1.0
- link motor_front_rightR_link: geometry collision cylinder length=0.021 radius=0.0425; visual mesh filename=package://minitaur_description/meshes/tmotor3.obj scale=1.0 1.0 1.0

File: minitaur_description/urdf/minitaur.urdf.xacro (robot description, xacro)
@@ -437,5 +437,5 @@
 			<visual>
 				<geometry>
-					<mesh filename="package://minitaur_description/urdf/tmotor3.obj" scale="1.0 1.0 1.0"/>
+					<mesh filename="package://minitaur_description/meshes/tmotor3.obj" scale="1.0 1.0 1.0"/>
 				</geometry>
 				<material name="motor"/>

File: minitaur_description/urdf/minitaur_gazebo.urdf (robot description, URDF)
Before this commit: robot minitaur, 40 links, 39 joints
Links:
- link motor_back_leftL_link: geometry collision cylinder length=0.021 radius=0.0425; visual mesh filename=model://minitaur_constrained/../../meshes/tmotor3.dae scale=100 100 100
- link motor_back_leftR_link: geometry collision cylinder length=0.021 radius=0.0425; visual mesh filename=model://minitaur_constrained/../../meshes/tmotor3.dae scale=100 100 100
- link motor_back_rightL_link: geometry collision cylinder length=0.021 radius=0.0425; visual mesh filename=model://minitaur_constrained/../../meshes/tmotor3.dae scale=100 100 100
- link motor_back_rightR_link: geometry collision cylinder length=0.021 radius=0.0425; visual mesh filename=model://minitaur_constrained/../../meshes/tmotor3.dae scale=100 100 100
- link motor_front_leftL_link: geometry collision cylinder length=0.021 radius=0.0425; visual mesh filename=model://minitaur_constrained/../../meshes/tmotor3.dae scale=100 100 100
- link motor_front_leftR_link: geometry collision cylinder length=0.021 radius=0.0425; visual mesh filename=model://minitaur_constrained/../../meshes/tmotor3.dae scale=100 100 100
- link motor_front_rightL_link: geometry collision cylinder length=0.021 radius=0.0425; visual mesh filename=model://minitaur_constrained/../../meshes/tmotor3.dae scale=100 100 100
- link motor_front_rightR_link: geometry collision cylinder length=0.021 radius=0.0425; visual mesh filename=model://minitaur_constrained/../../meshes/tmotor3.dae scale=100 100 100

File: minitaur_description/urdf/minitaur_gazebo.urdf.xacro (robot description, xacro)
@@ -510,5 +510,5 @@
 			<visual>
 				<geometry>
-					<mesh filename="model://minitaur_constrained/../../urdf/tmotor3.dae" scale="100 100 100"/>
+					<mesh filename="model://minitaur_constrained/../../meshes/tmotor3.dae" scale="100 100 100"/>
 				</geometry>
 			</visual>
