Commit message: Fixed dae description

File: minitaur_description/urdf/minitaur_gazebo.urdf (robot description, URDF)
Before this commit: robot minitaur, 40 links, 39 joints
Links:
- link motor_back_leftL_link: geometry collision cylinder length=0.021 radius=0.0425; visual mesh filename=model://minitaur_constrained/../../urdf/tmotor3.dae scale=100 100 100
- link motor_back_leftR_link: geometry collision cylinder length=0.021 radius=0.0425; visual mesh filename=model://minitaur_constrained/../../urdf/tmotor3.dae scale=100 100 100
- link motor_back_rightL_link: geometry collision cylinder length=0.021 radius=0.0425; visual mesh filename=model://minitaur_constrained/../../urdf/tmotor3.dae scale=100 100 100
- link motor_back_rightR_link: geometry collision cylinder length=0.021 radius=0.0425; visual mesh filename=model://minitaur_constrained/../../urdf/tmotor3.dae scale=100 100 100
- link motor_front_leftL_link: geometry collision cylinder length=0.021 radius=0.0425; visual mesh filename=model://minitaur_constrained/../../urdf/tmotor3.dae scale=100 100 100
- link motor_front_leftR_link: geometry collision cylinder length=0.021 radius=0.0425; visual mesh filename=model://minitaur_constrained/../../urdf/tmotor3.dae scale=100 100 100
- link motor_front_rightL_link: geometry collision cylinder length=0.021 radius=0.0425; visual mesh filename=model://minitaur_constrained/../../urdf/tmotor3.dae scale=100 100 100
- link motor_front_rightR_link: geometry collision cylinder length=0.021 radius=0.0425; visual mesh filename=model://minitaur_constrained/../../urdf/tmotor3.dae scale=100 100 100

File: minitaur_description/urdf/minitaur_gazebo.urdf.xacro (robot description, xacro)
@@ -510,5 +510,5 @@
 			<visual>
 				<geometry>
-					<mesh filename="/home/vasilisvasilop/catkin_ws/src/ghost_gazebo/minitaur_description/urdf/tmotor3.dae" scale="100 100 100"/>
+					<mesh filename="model://minitaur_constrained/../../urdf/tmotor3.dae" scale="100 100 100"/>
 				</geometry>
 			</visual>

Commit message: Fixed leg length

File: minitaur_description/urdf/minitaur_gazebo.urdf (robot description, URDF)
Before this commit: robot minitaur, 40 links, 39 joints
Links:
- link lower_leg_back_leftL_link: geometry collision box size=0.017 0.009 0.22; visual box size=0.017 0.009 0.22
- link lower_leg_back_rightR_link: geometry collision box size=0.017 0.009 0.22; visual box size=0.017 0.009 0.22
- link lower_leg_front_leftL_link: geometry collision box size=0.017 0.009 0.22; visual box size=0.017 0.009 0.22
- link lower_leg_front_rightR_link: geometry collision box size=0.017 0.009 0.22; visual box size=0.017 0.009 0.22
Joints:
- joint toe0: origin xyz=0 0 0.248 -> xyz=0 0 0.22
- joint toe2: origin xyz=0 0 0.248 -> xyz=0 0 0.22
- joint toe5: origin xyz=0 0 0.248 -> xyz=0 0 0.22
- joint toe7: origin xyz=0 0 0.248 -> xyz=0 0 0.22

File: minitaur_description/urdf/minitaur_gazebo.urdf.xacro (robot description, xacro)
@@ -57,5 +57,5 @@
 	<xacro:property name="lowerLegHeight" value="0.009"/>
 	<xacro:property name="lowerLegLength" value="0.2"/>
-	<xacro:property name="lowerLegLengthToe" value="0.248"/>
+	<xacro:property name="lowerLegLengthToe" value="0.22"/>
 	<xacro:property name="toeRadius" value="0.015"/>
 	<xacro:property name="toeStiffness" value="30000.0"/>
