Commit message: Modified friction properties

File: other/objects_description/caster_stool/caster_stool.urdf.xacro (robot description, xacro)
@@ -88,5 +88,5 @@
     <child link="caster_wheel" />
     <axis xyz="0 1 0"/>
-    <dynamics damping="0.01"/>
+    <dynamics damping="0.004"/>
   </joint>
 </robot>
