Commit message: Modified some friction parameters

File: other/objects_description/caster_cart/caster_cart.urdf.xacro (robot description, xacro)
@@ -88,5 +88,5 @@
     <child link="caster_wheel" />
     <axis xyz="0 1 0"/>
-    <dynamics damping="0.004"/>
+    <dynamics damping="0.04"/>
   </joint>
 </robot>

File: other/objects_description/caster_stool/caster_stool.urdf.xacro (robot description, xacro)
@@ -88,5 +88,5 @@
     <child link="caster_wheel" />
     <axis xyz="0 1 0"/>
-    <dynamics damping="0.001"/>
+    <dynamics damping="0.01"/>
   </joint>
 </robot>

Commit message: Added new world files

File: other/objects_description/caster_cart/caster_cart.urdf.xacro (robot description, xacro)
@@ -88,5 +88,5 @@
     <child link="caster_wheel" />
     <axis xyz="0 1 0"/>
-    <dynamics damping="0.04"/>
+    <dynamics damping="0.02"/>
   </joint>
 </robot>
